File: gp-ldo-test-board.sch (KiCad schematic (older format))
At the start: 6 parts

Commit message: initial schematic draft
Parts:
- added C? (x5): 4.7uF, symbol Device:C
- added C? (x2): DNP, symbol Device:C
- added C? (x2): 0.1uF, symbol Device:C
- added D? (x10): LED_Small, symbol Device:LED_Small
- added J? (x2): Conn_01x06, symbol Connector_Generic:Conn_01x06
- added J?: Conn_01x02, symbol Connector_Generic:Conn_01x02
- added JP? (x4): SolderJumper_2_Open, symbol Jumper:SolderJumper_2_Open
- added Q?: Q_PMOS_GDS, symbol Device:Q_PMOS_GDS
- added R? (x3): 10k, symbol Device:R_Small
- added R? (x2): DNP, symbol Device:R_Small
- added R? (x10): R_Small, symbol Device:R_Small
- added TP? (x7): TestPoint, symbol Connector:TestPoint
- added U? (x2): SLG46582, symbol gp-ldo-test-board:SLG46582
Connections:
- net labels added: AUX_LED_0, AUX_LED_1, LDO_VIN_SW, SLG0_SCL, SLG0_SDA, SLG1_SCL, SLG1_SDA, V_1.8_Vcore_FAULT, V_3.3_MGMT_FAULT, V_Vccio1_FAULT, V_Vccio2_FAULT
- wire segments 20 -> 196
Other:
- note added: "Silego never answered my question asking about \ndatasheet ambiguity here with Vih"
- note added: "aux LEDs here because other part\nneeds to control delayed power\non functionality"
- note added: "blinkenlights"
- note added: "for clipping scope probes"
- note added: "io0/io8 chosen to maximize\nchoice for analog pins"
- note added: "io3 chosen due to fewest\nalt uses (no OE)"
- note added: "latched fault indicators"
- note added: "testme: can caps be combined?"
- note added: "this is used for errata workaround"
- note added: "this will be used for link status\n(io expander) in the real design"
- note added: "unsure if parts will interfere with each other\nif programming only one of them"
- moved on the sheet: J?

Commit message: fix series resistors on ldos
Parts:
- added R? (x2): R_Small, symbol Device:R_Small
- C?: value 4.7uF -> DNP 4.7uF
- C? (x2): value DNP -> 2.2uF
Connections:
- wire segments 196 -> 198
Other:
- note added: "aux LEDs here because other part\nneeds to control delayed power\non functionality (design partitioning)"
- note added: "fixme: can caps be combined in any way?"
- note added: "fixme: do we even need these?"
- note added: "io3 chosen due to fewest\nalt uses (e.g. no OE/ACMP)"
- note added: "these resistors are needed because these slg\nparts are very power dissipation limited.\nthis hack is recommended by the datasheet"
- note added: "this is used for errata workaround\nto prevent voltage spikes on ldo outputs"
- note removed: "aux LEDs here because other part\nneeds to control delayed power\non functionality"
- note removed: "io3 chosen due to fewest\nalt uses (no OE)"
- note removed: "testme: can caps be combined?"
- note removed: "this is used for errata workaround"
Changed lines of the file:
@@
 Text Label 10650 3200 0    50   ~ 0
 V_Vccio2
-$Comp
-L Device:Q_PMOS_GDS Q?
-U 1 1 5F1212DA
-P 7500 1300
-F 0 "Q?" V 7749 1300 50  0000 C CNN
-F 1 "Q_PMOS_GDS" V 7840 1300 50  0000 C CNN
-F 2 "" H 7700 1400 50  0001 C CNN
-F 3 "~" H 7500 1300 50  0001 C CNN
-	1    7500 1300
-	0    1    1    0
-$EndComp
-Wire Wire Line
-	7700 1400 8100 1400
-Wire Wire Line
-	9500 1400 9500 2300
+Wire Wire Line
+	9500 1400 9500 2000
 Wire Wire Line
 	9600 2400 9600 2300
 Wire Wire Line
-	9600 2300 9500 2300
-Connection ~ 9500 2300
-Wire Wire Line
-	9500 2300 9500 2400
+	9500 2200 9500 2300
 Wire Wire Line
 	5900 2500 5900 2400
@@
 	5900 2400 6600 2400
 Wire Wire Line
-	8600 2400 8600 1400
+	8600 2400 8600 2300
 Connection ~ 8600 1400
 Wire Wire Line
@@
 	5800 2400 5900 2400
 Connection ~ 5900 2400
-$Comp
-L Device:C C?
-U 1 1 5F137485
-P 8100 1550
-F 0 "C?" H 8215 1596 50  0000 L CNN
-F 1 "4.7uF" H 8215 1505 50  0000 L CNN
-F 2 "" H 8138 1400 50  0001 C CNN
-F 3 "~" H 8100 1550 50  0001 C CNN
-	1    8100 1550
-	1    0    0    -1
-$EndComp
-Connection ~ 8100 1400
 Wire Wire Line
 	8100 1400 8600 1400
@@
 	1    0    0    -1
 $EndComp
-$Comp
-L Device:C C?
-U 1 1 5F13DF41
-P 6600 2550
-F 0 "C?" H 6715 2596 50  0000 L CNN
-F 1 "DNP" H 6715 2505 50  0000 L CNN
-F 2 "" H 6638 2400 50  0001 C CNN
-F 3 "~" H 6600 2550 50  0001 C CNN
-	1    6600 2550
-	1    0    0    -1
-$EndComp
 Connection ~ 6600 2400
 Wire Wire Line
@@
 	1    0    0    -1
 $EndComp
-Text Notes 6300 2200 0    50   ~ 0
-testme: can caps be combined?
+Text Notes 6150 2350 0    50   ~ 0
+fixme: can caps be combined in any way?
 $Comp
 L Device:C C?
@@
 P 10300 2450
 F 0 "C?" H 10415 2496 50  0000 L CNN
-F 1 "DNP" H 10415 2405 50  0000 L CNN
+F 1 "2.2uF" H 10415 2405 50  0000 L CNN
 F 2 "" H 10338 2300 50  0001 C CNN
 F 3 "~" H 10300 2450 50  0001 C CNN
@@
 	1    0    0    -1
 $EndComp
-$Comp
-L power:+5V #PWR?
-U 1 1 5F15221C
-P 7200 700
-F 0 "#PWR?" H 7200 550 50  0001 C CNN
-F 1 "+5V" H 7215 873 50  0000 C CNN
-F 2 "" H 7200 700 50  0001 C CNN
-F 3 "" H 7200 700 50  0001 C CNN
-	1    7200 700
-	1    0    0    -1
-$EndComp
-Wire Wire Line
-	7300 1400 7200 1400
-Wire Wire Line
-	7200 1400 7200 1000
-Text Notes 6550 1800 0    50   ~ 0
-this is used for errata workaround
-$Comp
-L Device:R_Small R?
-U 1 1 5F16257B
-P 7350 1000
-F 0 "R?" V 7154 1000 50  0000 C CNN
-F 1 "10k" V 7245 1000 50  0000 C CNN
-F 2 "" H 7350 1000 50  0001 C CNN
-F 3 "~" H 7350 1000 50  0001 C CNN
-	1    7350 1000
-	0    1    1    0
-$EndComp
-Wire Wire Line
-	7250 1000 7200 1000
-Connection ~ 7200 1000
-Wire Wire Line
-	7200 1000 7200 700
-Wire Wire Line
-	7450 1000 7500 1000
-Wire Wire Line
-	7500 1000 7500 1100
-Wire Wire Line
-	7500 1000 8100 1000
-Connection ~ 7500 1000
-Text Label 7600 1000 0    50   ~ 0
-LDO_VIN_SW
+Text Notes 6200 1900 0    50   ~ 0
+this is used for errata workaround\nto prevent voltage spikes on ldo outputs
 Wire Wire Line
 	5000 3500 4200 3500
@@
 V_Vccio2_FAULT
 Text Notes 4000 3000 0    50   ~ 0
-io3 chosen due to fewest\nalt uses (no OE)
+io3 chosen due to fewest\nalt uses (e.g. no OE/ACMP)
 Text Notes 2500 4100 0    50   ~ 0
 io0/io8 chosen to maximize\nchoice for analog pins
@@
 AUX_LED_1
 Text Notes 9850 4900 0    50   ~ 0
-aux LEDs here because other part\nneeds to control delayed power\non functionality
+aux LEDs here because other part\nneeds to control delayed power\non functionality (design partitioning)
 $Comp
 L Device:R_Small R?
@@
 Text Notes 13150 7350 0    50   ~ 0
 latched fault indicators
+$Comp
+L Device:C C?
+U 1 1 5F13DF41
+P 6600 2550
+F 0 "C?" H 6715 2596 50  0000 L CNN
+F 1 "2.2uF" H 6715 2505 50  0000 L CNN
+F 2 "" H 6638 2400 50  0001 C CNN
+F 3 "~" H 6600 2550 50  0001 C CNN
+	1    6600 2550
+	1    0    0    -1
+$EndComp
+$Comp
+L Device:C C?
+U 1 1 5F137485
+P 8100 1550
+F 0 "C?" H 8215 1596 50  0000 L CNN
+F 1 "DNP 4.7uF" H 8215 1505 50  0000 L CNN
+F 2 "" H 8138 1400 50  0001 C CNN
+F 3 "~" H 8100 1550 50  0001 C CNN
+	1    8100 1550
+	1    0    0    -1
+$EndComp
+Text Label 7600 1000 0    50   ~ 0
+LDO_VIN_SW
+Connection ~ 7500 1000
+Wire Wire Line
+	7500 1000 8100 1000
+Wire Wire Line
+	7500 1000 7500 1100
+Wire Wire Line
+	7450 1000 7500 1000
+Wire Wire Line
+	7200 1000 7200 700
+Connection ~ 7200 1000
+Wire Wire Line
+	7250 1000 7200 1000
+$Comp
+L Device:R_Small R?
+U 1 1 5F16257B
+P 7350 1000
+F 0 "R?" V 7154 1000 50  0000 C CNN
+F 1 "10k" V 7245 1000 50  0000 C CNN
+F 2 "" H 7350 1000 50  0001 C CNN
+F 3 "~" H 7350 1000 50  0001 C CNN
+	1    7350 1000
+	0    1    1    0
+$EndComp
+Wire Wire Line
+	7200 1400 7200 1000
+Wire Wire Line
+	7300 1400 7200 1400
+$Comp
+L power:+5V #PWR?
+U 1 1 5F15221C
+P 7200 700
+F 0 "#PWR?" H 7200 550 50  0001 C CNN
+F 1 "+5V" H 7215 873 50  0000 C CNN
+F 2 "" H 7200 700 50  0001 C CNN
+F 3 "" H 7200 700 50  0001 C CNN
+	1    7200 700
+	1    0    0    -1
+$EndComp
+$Comp
+L Device:Q_PMOS_GDS Q?
+U 1 1 5F1212DA
+P 7500 1300
+F 0 "Q?" V 7749 1300 50  0000 C CNN
+F 1 "Q_PMOS_GDS" V 7840 1300 50  0000 C CNN
+F 2 "" H 7700 1400 50  0001 C CNN
+F 3 "~" H 7500 1300 50  0001 C CNN
+	1    7500 1300
+	0    1    1    0
+$EndComp
+Text Notes 3800 1900 0    50   ~ 0
+fixme: do we even need these?
+Connection ~ 8100 1400
+Wire Wire Line
+	7700 1400 8100 1400
+$Comp
+L Device:R_Small R?
+U 1 1 5F3C1459
+P 8600 2200
+F 0 "R?" H 8450 2250 50  0000 L CNN
+F 1 "R_Small" H 8200 2150 50  0000 L CNN
+F 2 "" H 8600 2200 50  0001 C CNN
+F 3 "~" H 8600 2200 50  0001 C CNN
+	1    8600 2200
+	1    0    0    -1
+$EndComp
+Wire Wire Line
+	8600 2100 8600 1400
+$Comp
+L Device:R_Small R?
+U 1 1 5F3C26A2
+P 9500 2100
+F 0 "R?" H 9550 2150 50  0000 L CNN
+F 1 "R_Small" H 9550 2050 50  0000 L CNN
+F 2 "" H 9500 2100 50  0001 C CNN
+F 3 "~" H 9500 2100 50  0001 C CNN
+	1    9500 2100
+	1    0    0    -1
+$EndComp
+Wire Wire Line
+	9600 2300 9500 2300
+Connection ~ 9500 2300
+Wire Wire Line
+	9500 2300 9500 2400
+Text Notes 9650 2050 0    50   ~ 0
+these resistors are needed because these slg\nparts are very power dissipation limited.\nthis hack is recommended by the datasheet
 $EndSCHEMATC

Commit message: footprints and initial place
Parts:
- removed C?: DNP 4.7uF, symbol Device:C
- removed Q?: Q_PMOS_GDS, symbol Device:Q_PMOS_GDS
- added Q1: Q_PMOS_GSD, Package_TO_SOT_SMD:SOT-23, symbol Device:Q_PMOS_GSD
- C1, C3: renamed from C?; footprint (none) -> Capacitor_SMD:C_0402_1005Metric
- C2, C4: renamed from C?; value 2.2uF -> 4.7uF; footprint (none) -> Capacitor_SMD:C_0805_2012Metric
- C5, C6, C7, C8: renamed from C?; footprint (none) -> Capacitor_SMD:C_0805_2012Metric
- D1, D2: renamed from D?; value LED_Small -> YELLOW; footprint (none) -> LED_SMD:LED_0805_2012Metric
- D10, D7, D8, D9: renamed from D?; value LED_Small -> RED; footprint (none) -> LED_SMD:LED_0805_2012Metric
- D3, D4, D5, D6: renamed from D?; value LED_Small -> GREEN; footprint (none) -> LED_SMD:LED_0805_2012Metric
- J1: renamed from J?; footprint (none) -> Connector_PinHeader_2.54mm:PinHeader_1x03_P2.54mm_Vertical
- J2, J4, J6, J7, J8, J9: renamed from J?; footprint (none) -> Connector_PinHeader_2.54mm:PinHeader_1x02_P2.54mm_Vertical
- J3, J5: renamed from J?; footprint (none) -> Connector_PinHeader_2.54mm:PinHeader_1x06_P2.54mm_Vertical
- JP1, JP2, JP3, JP4: renamed from JP?; footprint (none) -> Jumper:SolderJumper-2_P1.3mm_Open_Pad1.0x1.5mm
- R1, R2, R3, R4, R6: renamed from R?; footprint (none) -> Resistor_SMD:R_0402_1005Metric
- R10, R11, R12, R13, R14, R15, R16, R17, R7, R8: renamed from R?; value R_Small -> 1k; footprint (none) -> Resistor_SMD:R_0402_1005Metric
- R5, R9: renamed from R?; value R_Small -> 2.2; footprint (none) -> Resistor_SMD:R_0402_1005Metric
- TP1, TP2, TP3, TP4, TP5, TP6, TP7: renamed from TP?; footprint (none) -> TestPoint:TestPoint_Pad_1.0x1.0mm
- U1, U2: renamed from U?; footprint (none) -> gp-ldo-test-board:SLG46580
Connections:
- wire segments 198 -> 197
Other:
- note removed: "fixme: can caps be combined in any way?"
- moved on the sheet: R5
