File: gp-ldo-test-board.kicad_pcb (KiCad board)
At the start: 2 copper layers, 38.1 x 25.4 mm, 58 parts, among them J1 Conn_01x03, J2 Conn_01x02, J3 Conn_01x06, J4 Conn_01x02, J5 Conn_01x06, J6 Conn_01x02, J7 Conn_01x02, J8 Conn_01x02, J9 Conn_01x02, Q1 Q_PMOS_GSD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

Commit message: tweaks
Routing:
- net /V_Vccio1_FAULT: track 14.8 -> 23.3 mm
- net GND: track 44.8 -> 42.4 mm
- net /V_Vccio2_FAULT: track 13.8 -> 15.0 mm
- net Net-(J5-Pad5): track 13.9 -> 14.0 mm, vias 0 -> 2
Other:
- board text added: "UwU"
